File: rf/2stage_qpl_lna/2stage_qpl_lna.kicad_sch (KiCad schematic)
At the start: 25 parts, among them J1 SMA, J2 EXT_PWR, J3 SMA, U1 QPL9547, U2 QPL9547, X1 SAW, X2 SAW

Commit message: Update QPL based LNA
Parts:
- D1: footprint LED_THT:LED_D5.0mm_Clear -> LED_SMD:LED_0603_1608Metric; MFR (none) -> 859-LTST-C190GKT
Changed lines of the file:
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@@
 			)
 		)
-		(property "Footprint" "LED_THT:LED_D5.0mm_Clear"
+		(property "Footprint" "LED_SMD:LED_0603_1608Metric"
 			(at 59.69 149.86 0)
 			(effects
@@
 			(at 59.69 149.86 0)
 			(effects
+				(font
+					(size 1.27 1.27)
+				)
+				(hide yes)
+			)
+		)
+		(property "MFR" "859-LTST-C190GKT"
+			(at 59.69 149.86 0)
+			(effects
