File: rf/L_band_backfire_lna/L_band_backfire_lna.kicad_sch (KiCad schematic)
At the start: 24 parts, among them J1 SMA, J2 SMA, U1 QPL9547, U2 QPL9547, X1 SAW, X2 SAW

Commit message: Diameter =/= Radius dum dum
Parts:
- J1: footprint TestPoint:TestPoint_THTPad_D4.0mm_Drill2.0mm -> Connector_Pin:Pin_D1.3mm_L11.0mm_LooseFit
Changed lines of the file:
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@@
 			)
 		)
-		(property "Footprint" "TestPoint:TestPoint_THTPad_D4.0mm_Drill2.0mm"
+		(property "Footprint" "Connector_Pin:Pin_D1.3mm_L11.0mm_LooseFit"
 			(at 66.04 97.79 0)
 			(effects

Commit message: owo what's that :3
Parts:
- J1: footprint Connector_Pin:Pin_D1.3mm_L11.0mm_LooseFit -> Special_hole:Special Hole
Changed lines of the file:
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@@
 			)
 		)
-		(property "Footprint" "Connector_Pin:Pin_D1.3mm_L11.0mm_LooseFit"
+		(property "Footprint" "Special_hole:Special Hole"
 			(at 66.04 97.79 0)
 			(effects
